File: scaffold/scaffold.kicad_pcb (KiCad board)
At the start: 2 copper layers, 242 x 155 mm, 34 parts, among them SW1 SW_Push, SW2 SW_Push, U1 Pro_Micro, U2 Pro_Micro

Commit message: Scaffold V2: wider spacing for supports for better switch fit, updated assembly guide.
Parts:
- removed the G*** at (141.0, 88.9)
- removed the G*** at (102.8, 81.9)
- added G***: LOGO, scaffold:scaffold_logo, F.Cu at (102.6, 81.9)
- added G***: LOGO, scaffold:scaffold_logo, F.Cu at (140.8, 88.9)
- Col1, Col5, ColR1, ColR5: footprint scaffold:Col3_socket_PG1350_sod123_cutouts -> scaffold:Col3_socket_PG1350_sod123_cutouts_v2
- Col2, Col3, Col4, ColR2, ColR3, ColR4: footprint scaffold:Col4_socket_PG1350_sod123_cutouts -> scaffold:Col4_socket_PG1350_sod123_cutouts_v2
- SW_and_D1, SW_and_D2, SW_and_D3, SW_and_DR1, SW_and_DR2, SW_and_DR3: footprint scaffold:Col1_socket_PG1350_sod123_cutouts -> scaffold:Col1_socket_PG1350_sod123_cutouts_v2
- moved J_TRRS_1 27.0 mm to (5.65, 45.2)
- moved J_TRRS_2 27.0 mm to (236.3, 45.2)
- moved Joycon_thumb2 3.22 mm to (165.4, 46.4)
- moved Joycon_thumb1 2.02 mm to (99.8, 58.0)
- moved SW1 1.50 mm to (30.4, 15.4)
- moved SW2 1.50 mm to (205.1, 15.4)
Routing:
- net /COL_M: track 155.5 -> 199.7 mm
- net /COL_RT: track 128.8 -> 166.1 mm, vias 5 -> 4
- net /COL_R: track 190.4 -> 224.3 mm, vias 4 -> 3
- net /COL_RR: track 238.6 -> 270.3 mm
- net /COL_I1: track 140.4 -> 172.1 mm
- net /COL_P: track 216.7 -> 242.3 mm
- net /COL_RI1: track 150.2 -> 174.5 mm
- net /COL_RM: track 211.3 -> 234.4 mm
- net /ROW_RT: track 356.3 -> 377.0 mm
- net /COL_RP: track 227.0 -> 247.2 mm
- net /COL_T: track 159.9 -> 179.7 mm, vias 5 -> 4
- net /COL_I2: track 86.9 -> 106.4 mm
- net +5V: track 97.0 -> 114.3 mm, vias 1 -> 2
- net /ROW_T: track 355.8 -> 340.9 mm
- net /SERIAL: track 7.57 -> 20.5 mm
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Other:
- outline, holes or cut-outs redrawn
